Commit message: urdf

File: robot_ws/src/nsra_support/urdf/Robot.urdf (robot description, URDF)
Before this commit: robot None, 0 links, 0 joints
Links:
- added link Component1_1, mass 20.922358; collision mesh filename=package://fusion2urdf/Robot/bin_stl/Component1_1_m-binary.s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; visual mesh filename=package://fusion2urdf/Robot/bin_stl/Component1_1_m-binary.s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
- added link Component2_1, mass 13.1521; collision mesh filename=package://fusion2urdf/Robot/bin_stl/Component2_1_m-binary.s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; visual mesh filename=package://fusion2urdf/Robot/bin_stl/Component2_1_m-binary.s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
- added link Component3_1, mass 11.720524; collision mesh filename=package://fusion2urdf/Robot/bin_stl/Component3_1_m-binary.s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; visual mesh filename=package://fusion2urdf/Robot/bin_stl/Component3_1_m-binary.s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
- added link Component4_1, mass 3.348314; collision mesh filename=package://fusion2urdf/Robot/bin_stl/Component4_1_m-binary.s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; visual mesh filename=package://fusion2urdf/Robot/bin_stl/Component4_1_m-binary.s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
- added link Component5_1, mass 2.858845; collision mesh filename=package://fusion2urdf/Robot/bin_stl/Component5_1_m-binary.s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; visual mesh filename=package://fusion2urdf/Robot/bin_stl/Component5_1_m-binary.s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
- added link Component6_1, mass 0.340558; collision mesh filename=package://fusion2urdf/Robot/bin_stl/Component6_1_m-binary.s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; visual mesh filename=package://fusion2urdf/Robot/bin_stl/Component6_1_m-binary.s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
- added link base_link, mass 205.712105; collision mesh filename=package://fusion2urdf/Robot/bin_stl/base_link_m-binary.stl; visual mesh filename=package://fusion2urdf/Robot/bin_stl/base_link_m-binary.stl
Joints:
- added joint Rev1: type revolute, parent base_link, child Component1_1, origin xyz=0.2 -0.366257 0.0 rpy=0 0 0, axis 0.0 0.01 0.0, limit lower=-2.0944 upper=2.0944 effort=1 velocity=1.0
- added joint Rev2: type revolute, parent Component1_1, child Component2_1, origin xyz=0.0 0.151 -0.1276 rpy=0 0 0, axis 0.0 -0.0 0.01, limit lower=-1.5708 upper=1.5708 effort=1 velocity=1.0
- added joint Rev3: type revolute, parent Component2_1, child Component3_1, origin xyz=0.0 0.459999 0.1741 rpy=0 0 0, axis 0.0 -0.0 0.01, limit lower=-1.5708 upper=1.5708 effort=1 velocity=1.0
- added joint Rev4: type revolute, parent Component3_1, child Component4_1, origin xyz=0.015 0.106 -0.0465 rpy=0 0 0, axis 0.01 0.0 -0.0, limit lower=-3.1415 upper=3.1415 effort=1 velocity=1.0
- added joint Rev5: type revolute, parent Component4_1, child Component5_1, origin xyz=0.426 0.0 0.04 rpy=0 0 0, axis 0.0 -0.0 0.01, limit lower=-1.7453 upper=1.7453 effort=1 velocity=1.0
- added joint Rev6: type continuous, parent Component5_1, child Component6_1, origin xyz=0.052 0.0 -0.04 rpy=0 0 0, axis 0.01 -0.0 -0.0
