Commit message: Update nsra.xacro

File: robot_ws/src/nsra_support/urdf/nsra.xacro (robot description, xacro)
@@ -19,5 +19,5 @@
   <parent link="table"/>
   <child link="base_link"/>
-  <origin xyz="0 0 0.9" rpy="1.5708 0 0"/>
+  <origin xyz="0 0 0.9" rpy="0 0 0"/>
 </joint>
 </robot>

Commit message: Update nsra.xacro

File: robot_ws/src/nsra_support/urdf/nsra.xacro (robot description, xacro)
@@ -9,5 +9,5 @@
   <parent link="world"/>
   <child link="table"/>
-  <origin xyz="0 0 0" rpy="0 0 0"/>
+  <origin xyz="0 0 0" rpy="1.5708 0 0"/>
 </joint>
 <joint name="world_to_camera" type="fixed">

Commit message: tf

File: robot_ws/src/nsra_support/urdf/nsra.xacro (robot description, xacro)
@@ -9,5 +9,5 @@
   <parent link="world"/>
   <child link="table"/>
-  <origin xyz="0 0 0" rpy="1.5708 0 0"/>
+  <origin xyz="0 0 0" rpy="0 0 0"/>
 </joint>
 <joint name="world_to_camera" type="fixed">

File: robot_ws/src/nsra_support/urdf/robot.xacro (robot description, xacro)
@@ -4,5 +4,5 @@
 <link name="base_link">
   <inertial>
-    <origin rpy="0 0 0" xyz="0.198887 -0.80113 0.021369"/>
+    <origin rpy="1.5708 0 0" xyz="0.198887 -0.80113 0.021369"/>
     <mass value="204.473744"/>
     <inertia ixx="6.821919" ixy="0.014918" ixz="4.362239" iyy="13.382202" iyz="-4.356184" izz="7.679036"/>

Commit message: Update nsra.xacro

File: robot_ws/src/nsra_support/urdf/nsra.xacro (robot description, xacro)
@@ -19,5 +19,5 @@
   <parent link="table"/>
   <child link="base_link"/>
-  <origin xyz="0 0 0.9" rpy="0 0 0"/>
+  <origin xyz="0 0 0.9" rpy="1.5708 0 0"/>
 </joint>
 </robot>

Commit message: Update nsra.xacro

File: robot_ws/src/nsra_support/urdf/nsra.xacro (robot description, xacro)
@@ -19,5 +19,5 @@
   <parent link="table"/>
   <child link="base_link"/>
-  <origin xyz="0 0 0.9" rpy="1.5708 0 0"/>
+  <origin xyz="0 0 0" rpy="1.5708 0 0"/>
 </joint>
 </robot>

Commit message: Update nsra.xacro

File: robot_ws/src/nsra_support/urdf/nsra.xacro (robot description, xacro)
@@ -19,5 +19,5 @@
   <parent link="table"/>
   <child link="base_link"/>
-  <origin xyz="0 0 0" rpy="1.5708 0 0"/>
+  <origin xyz="0 0.2 0.9" rpy="1.5708 0 0"/>
 </joint>
 </robot>

Commit message: Update nsra.xacro

File: robot_ws/src/nsra_support/urdf/nsra.xacro (robot description, xacro)
@@ -19,5 +19,5 @@
   <parent link="table"/>
   <child link="base_link"/>
-  <origin xyz="0 0.2 0.9" rpy="1.5708 0 0"/>
+  <origin xyz="0.2 0.4 0.9" rpy="1.5708 0 0"/>
 </joint>
 </robot>

Commit message: Update nsra.xacro

File: robot_ws/src/nsra_support/urdf/nsra.xacro (robot description, xacro)
@@ -19,5 +19,5 @@
   <parent link="table"/>
   <child link="base_link"/>
-  <origin xyz="0.2 0.4 0.9" rpy="1.5708 0 0"/>
+  <origin xyz="0.1 0.3 0.9" rpy="1.5708 0 0"/>
 </joint>
 </robot>

Commit message: Update nsra.xacro

File: robot_ws/src/nsra_support/urdf/nsra.xacro (robot description, xacro)
@@ -19,5 +19,5 @@
   <parent link="table"/>
   <child link="base_link"/>
-  <origin xyz="0.1 0.3 0.9" rpy="1.5708 0 0"/>
+  <origin xyz="0.075 0.275 0.9" rpy="1.5708 0 0"/>
 </joint>
 </robot>

Commit message: Update nsra.xacro

File: robot_ws/src/nsra_support/urdf/nsra.xacro (robot description, xacro)
@@ -19,5 +19,5 @@
   <parent link="table"/>
   <child link="base_link"/>
-  <origin xyz="0.075 0.275 0.9" rpy="1.5708 0 0"/>
+  <origin xyz="0.07505 0.275 0.905" rpy="1.5708 0 0"/>
 </joint>
 </robot>

Commit message: Update nsra.xacro

File: robot_ws/src/nsra_support/urdf/nsra.xacro (robot description, xacro)
@@ -19,5 +19,5 @@
   <parent link="table"/>
   <child link="base_link"/>
-  <origin xyz="0.07505 0.275 0.905" rpy="1.5708 0 0"/>
+  <origin xyz="0.07605 0.276 0.905" rpy="1.5708 0 0"/>
 </joint>
 </robot>

Commit message: Update nsra.xacro

File: robot_ws/src/nsra_support/urdf/nsra.xacro (robot description, xacro)
@@ -19,5 +19,5 @@
   <parent link="table"/>
   <child link="base_link"/>
-  <origin xyz="0.07605 0.276 0.905" rpy="1.5708 0 0"/>
+  <origin xyz="0.08005 0.280 0.905" rpy="1.5708 0 0"/>
 </joint>
 </robot>

Commit message: Update nsra.xacro

File: robot_ws/src/nsra_support/urdf/nsra.xacro (robot description, xacro)
@@ -19,5 +19,5 @@
   <parent link="table"/>
   <child link="base_link"/>
-  <origin xyz="0.08005 0.280 0.905" rpy="1.5708 0 0"/>
+  <origin xyz="0.09005 0.290 0.905" rpy="1.5708 0 0"/>
 </joint>
 </robot>

Commit message: Update nsra.xacro

File: robot_ws/src/nsra_support/urdf/nsra.xacro (robot description, xacro)
@@ -19,5 +19,5 @@
   <parent link="table"/>
   <child link="base_link"/>
-  <origin xyz="0.09005 0.290 0.905" rpy="1.5708 0 0"/>
+  <origin xyz="0.07005 0.270 0.905" rpy="1.5708 0 0"/>
 </joint>
 </robot>

Commit message: Update nsra.xacro

File: robot_ws/src/nsra_support/urdf/nsra.xacro (robot description, xacro)
@@ -19,5 +19,5 @@
   <parent link="table"/>
   <child link="base_link"/>
-  <origin xyz="0.07005 0.270 0.905" rpy="1.5708 0 0"/>
+  <origin xyz="0.07005 0.270 0.9025" rpy="1.5708 0 0"/>
 </joint>
 </robot>

Commit message: Update nsra.xacro

File: robot_ws/src/nsra_support/urdf/nsra.xacro (robot description, xacro)
@@ -19,5 +19,5 @@
   <parent link="table"/>
   <child link="base_link"/>
-  <origin xyz="0.07005 0.270 0.9025" rpy="1.5708 0 0"/>
+  <origin xyz="0.07005 0.270 0.9045" rpy="1.5708 0 0"/>
 </joint>
 </robot>

Commit message: Update nsra.xacro

File: robot_ws/src/nsra_support/urdf/nsra.xacro (robot description, xacro)
@@ -19,5 +19,5 @@
   <parent link="table"/>
   <child link="base_link"/>
-  <origin xyz="0.07005 0.270 0.9045" rpy="1.5708 0 0"/>
+  <origin xyz="0 0 0" rpy="1.5708 0 0"/>
 </joint>
 </robot>

Commit message: Update nsra.xacro

File: robot_ws/src/nsra_support/urdf/nsra.xacro (robot description, xacro)
@@ -19,5 +19,5 @@
   <parent link="table"/>
   <child link="base_link"/>
-  <origin xyz="0 0 0" rpy="1.5708 0 0"/>
+  <origin xyz="0 0 0.5" rpy="1.5708 0 0"/>
 </joint>
 </robot>

Commit message: Update nsra.xacro

File: robot_ws/src/nsra_support/urdf/nsra.xacro (robot description, xacro)
@@ -19,5 +19,5 @@
   <parent link="table"/>
   <child link="base_link"/>
-  <origin xyz="0 0 0.5" rpy="1.5708 0 0"/>
+  <origin xyz="0 0 0.65" rpy="1.5708 0 0"/>
 </joint>
 </robot>

Commit message: Update nsra.xacro

File: robot_ws/src/nsra_support/urdf/nsra.xacro (robot description, xacro)
@@ -19,5 +19,5 @@
   <parent link="table"/>
   <child link="base_link"/>
-  <origin xyz="0 0 0.65" rpy="1.5708 0 0"/>
+  <origin xyz="0 0 0.6" rpy="1.5708 0 0"/>
 </joint>
 </robot>

Commit message: Update nsra.xacro

File: robot_ws/src/nsra_support/urdf/nsra.xacro (robot description, xacro)
@@ -19,5 +19,5 @@
   <parent link="table"/>
   <child link="base_link"/>
-  <origin xyz="0 0 0.6" rpy="1.5708 0 0"/>
+  <origin xyz="0.27 0 0.57" rpy="1.5708 0 0"/>
 </joint>
 </robot>

Commit message: Update nsra.xacro

File: robot_ws/src/nsra_support/urdf/nsra.xacro (robot description, xacro)
@@ -19,5 +19,5 @@
   <parent link="table"/>
   <child link="base_link"/>
-  <origin xyz="0.27 0 0.57" rpy="1.5708 0 0"/>
+  <origin xyz="0 0.27 0.5695" rpy="1.5708 0 0"/>
 </joint>
 </robot>

Commit message: Update nsra.xacro

File: robot_ws/src/nsra_support/urdf/nsra.xacro (robot description, xacro)
@@ -19,5 +19,5 @@
   <parent link="table"/>
   <child link="base_link"/>
-  <origin xyz="0 0.27 0.5695" rpy="1.5708 0 0"/>
+  <origin xyz="-0.7 0.27 0.5705" rpy="1.5708 0 0"/>
 </joint>
 </robot>

Commit message: Update nsra.xacro

File: robot_ws/src/nsra_support/urdf/nsra.xacro (robot description, xacro)
@@ -19,5 +19,5 @@
   <parent link="table"/>
   <child link="base_link"/>
-  <origin xyz="-0.7 0.27 0.5705" rpy="1.5708 0 0"/>
+  <origin xyz="-0.5 0.27 0.572" rpy="1.5708 0 0"/>
 </joint>
 </robot>

Commit message: Update nsra.xacro

File: robot_ws/src/nsra_support/urdf/nsra.xacro (robot description, xacro)
@@ -19,5 +19,5 @@
   <parent link="table"/>
   <child link="base_link"/>
-  <origin xyz="-0.5 0.27 0.572" rpy="1.5708 0 0"/>
+  <origin xyz="-0.42 0.27 0.574" rpy="1.5708 0 0"/>
 </joint>
 </robot>

Commit message: Update nsra.xacro

File: robot_ws/src/nsra_support/urdf/nsra.xacro (robot description, xacro)
@@ -19,5 +19,5 @@
   <parent link="table"/>
   <child link="base_link"/>
-  <origin xyz="-0.42 0.27 0.574" rpy="1.5708 0 0"/>
+  <origin xyz="-0.45 0.27 0.575" rpy="1.5708 0 0"/>
 </joint>
 </robot>

Commit message: Update nsra.xacro

File: robot_ws/src/nsra_support/urdf/nsra.xacro (robot description, xacro)
@@ -19,5 +19,5 @@
   <parent link="table"/>
   <child link="base_link"/>
-  <origin xyz="-0.45 0.27 0.575" rpy="1.5708 0 0"/>
+  <origin xyz="-0.47 0.27 0.576" rpy="1.5708 0 0"/>
 </joint>
 </robot>

Commit message: Update nsra.xacro

File: robot_ws/src/nsra_support/urdf/nsra.xacro (robot description, xacro)
@@ -19,5 +19,5 @@
   <parent link="table"/>
   <child link="base_link"/>
-  <origin xyz="-0.47 0.27 0.576" rpy="1.5708 0 0"/>
+  <origin xyz="-0.47 0.27 0.578" rpy="1.5708 0 0"/>
 </joint>
 </robot>

Commit message: Update nsra.xacro

File: robot_ws/src/nsra_support/urdf/nsra.xacro (robot description, xacro)
@@ -19,5 +19,5 @@
   <parent link="table"/>
   <child link="base_link"/>
-  <origin xyz="-0.47 0.27 0.578" rpy="1.5708 0 0"/>
+  <origin xyz="-0.47 0.27 0.58" rpy="1.5708 0 0"/>
 </joint>
 </robot>

Commit message: Update nsra.xacro

File: robot_ws/src/nsra_support/urdf/nsra.xacro (robot description, xacro)
@@ -19,5 +19,5 @@
   <parent link="table"/>
   <child link="base_link"/>
-  <origin xyz="-0.47 0.27 0.58" rpy="1.5708 0 0"/>
+  <origin xyz="-0.47 0.27 0.5795" rpy="1.5708 0 0"/>
 </joint>
 </robot>
