Commit message: Update robot.xacro

File: robot_ws/src/nsra_support/urdf/robot.xacro (robot description, xacro)
@@ -4,5 +4,5 @@
 <link name="base_link">
   <inertial>
-    <origin rpy="1.5708 0 0" xyz="0.198887 -0.80113 0.021369"/>
+    <origin rpy="0 0 0" xyz="0.198887 -0.80113 0.021369"/>
     <mass value="204.473744"/>
     <inertia ixx="6.821919" ixy="0.014918" ixz="4.362239" iyy="13.382202" iyz="-4.356184" izz="7.679036"/>

Commit message: Update robot.xacro

File: robot_ws/src/nsra_support/urdf/robot.xacro (robot description, xacro)
@@ -161,5 +161,5 @@
   <child link="Component2_1"/>
   <axis xyz="0.01 -0.0 -0.0"/>
-  <limit effort="30" velocity="1.0" lower="-2" upper="1" />
+  <limit effort="1" velocity="1.0" lower="-1.5708" upper="1.5708" />
 </joint>
 <transmission name="Rev2_tran">
@@ -178,5 +178,5 @@
   <child link="Component3_1"/>
   <axis xyz="-0.01 0.0 -0.0"/>
-  <limit effort="30" velocity="1.0" lower="-2.2" upper="0.7" />
+  <limit effort="1" velocity="1.0" lower="-1.5708" upper="1.5708" />
 </joint>
 <transmission name="Rev3_tran">
@@ -195,4 +195,5 @@
   <child link="Component4_1"/>
   <axis xyz="-0.0 -0.0 0.01"/>
+  <limit effort="1" velocity="1.0" lower="-3.1415" upper="3.1415" />
 </joint>
 <transmission name="Rev4_tran">
@@ -211,4 +212,5 @@
   <child link="Component5_1"/>
   <axis xyz="-0.01 0.0 0.0"/>
+  <limit effort="1" velocity="1.0" lower="-1.7453" upper="1.7453" />
 </joint>
 <transmission name="Rev5_tran">
@@ -243,4 +245,5 @@
   <child link="Component1_1"/>
   <axis xyz="0.0 0.01 0.0"/>
+  <limit effort="1" velocity="1.0" lower="-2.0944" upper="2.0944" />
 </joint>
 <transmission name="Rev1_tran">

Commit message: Update robot.xacro

File: robot_ws/src/nsra_support/urdf/robot.xacro (robot description, xacro)
@@ -156,5 +156,5 @@
   </collision>
 </link>
-<joint name="Rev2" type="continuous">
+<joint name="Rev2" type="revolute">
   <origin rpy="0 0 0" xyz="0.04741 0.151 0.0"/>
   <parent link="Component1_1"/>
@@ -173,5 +173,5 @@
   </actuator>
 </transmission>
-<joint name="Rev3" type="continuous">
+<joint name="Rev3" type="revolute">
   <origin rpy="0 0 0" xyz="-0.09391 0.46 0.0"/>
   <parent link="Component2_1"/>
@@ -190,5 +190,5 @@
   </actuator>
 </transmission>
-<joint name="Rev4" type="continuous">
+<joint name="Rev4" type="revolute">
   <origin rpy="0 0 0" xyz="0.0465 0.106 0.015"/>
   <parent link="Component3_1"/>
@@ -207,5 +207,5 @@
   </actuator>
 </transmission>
-<joint name="Rev5" type="continuous">
+<joint name="Rev5" type="revolute">
   <origin rpy="0 0 0" xyz="-0.04 0.0 0.481"/>
   <parent link="Component4_1"/>
@@ -240,5 +240,5 @@
   </actuator>
 </transmission>
-<joint name="Rev1" type="continuous">
+<joint name="Rev1" type="revolute">
   <origin rpy="0 0 0" xyz="0.2 -0.691257 0.0"/>
   <parent link="base_link"/>

Commit message: urdf

File: robot_ws/src/nsra_support/urdf/robot.xacro (robot description, xacro)
@@ -241,9 +241,10 @@
   </actuator>
 </transmission>
-<joint name="Rev6" type="continuous">
+<joint name="Rev6" type="revolute">
   <origin rpy="0 0 0" xyz="0.052 0.0 -0.04"/>
   <parent link="Component5_1"/>
   <child link="Component6_1"/>
   <axis xyz="0.01 -0.0 -0.0"/>
+  <limit effort="1" velocity="1.0" lower="-1.5708" upper="1.5708" />
 </joint>
 <transmission name="Rev6_tran">

Commit message: urdf

File: robot_ws/src/nsra_support/urdf/robot.xacro (robot description, xacro)
@@ -246,5 +246,5 @@
   <child link="Component6_1"/>
   <axis xyz="0.01 -0.0 -0.0"/>
-  <limit effort="1" velocity="1.0" lower="-1.5708" upper="1.5708" />
+  <limit effort="1" velocity="1.0" lower="-3.1415" upper="3.1415" />
 </joint>
 <transmission name="Rev6_tran">
