Commit message: Update robot.xacro

File: robot_ws/src/nsra_urdf/urdf/robot.xacro (robot description, xacro)
@@ -218,5 +218,5 @@
 </transmission>
 <joint name="Rev2" type="revolute">
-  <origin rpy="0 0 0" xyz="0.0 -0.059 -0.12679"/>
+  <origin rpy="0 0 0" xyz="0.0 0.151 -0.12679"/>
   <parent link="Component1_1"/>
   <child link="Component2_1"/>

Commit message: Update robot.xacro

File: robot_ws/src/nsra_urdf/urdf/robot.xacro (robot description, xacro)
@@ -48,10 +48,10 @@
 <link name="Component2_1">
   <inertial>
-    <origin rpy="0 0 0" xyz="0.0 0.436486 0.05349900000000002"/>
+    <origin rpy="0 0 0" xyz="0.0 0.226486 0.05349900000000002"/>
     <mass value="13.1521"/>
     <inertia ixx="0.673202" ixy="-0.0" ixz="-0.235485" iyy="0.032171" iyz="0.181962" izz="0.660051"/>
   </inertial>
   <visual>
-    <origin rpy="0 0 0" xyz="-0.2 0.425257 0.12679"/>
+    <origin rpy="0 0 0" xyz="-0.2 0.215257 0.12679"/>
     <geometry>
       <mesh filename="package://nsra_urdf/urdf/mm_stl/Component2_1.stl" scale="0.001 0.001 0.001"/>
@@ -62,5 +62,5 @@
   </visual>
   <collision>
-    <origin rpy="0 0 0" xyz="-0.2 0.425257 0.12679"/>
+    <origin rpy="0 0 0" xyz="-0.2 0.215257 0.12679"/>
     <geometry>
       <mesh filename="package://nsra_urdf/urdf/mm_stl/Component2_1.stl" scale="0.001 0.001 0.001"/>

Commit message: Update robot.xacro

File: robot_ws/src/nsra_urdf/urdf/robot.xacro (robot description, xacro)
@@ -235,5 +235,5 @@
 </transmission>
 <joint name="Rev3" type="revolute">
-  <origin rpy="0 0 0" xyz="0.0 0.67 0.1741"/>
+  <origin rpy="0 0 0" xyz="0.0 0.459999 0.1741"/>
   <parent link="Component2_1"/>
   <child link="Component3_1"/>

Commit message: Update robot.xacro

File: robot_ws/src/nsra_urdf/urdf/robot.xacro (robot description, xacro)
@@ -269,5 +269,5 @@
 </transmission>
 <joint name="Rev5" type="revolute">
-  <origin rpy="0 0 0" xyz="0.426 0.0 0.04"/>
+  <origin rpy="0 0 0" xyz="0.326 0.0 0.04"/>
   <parent link="Component4_1"/>
   <child link="Component5_1"/>

Commit message: Update robot.xacro

File: robot_ws/src/nsra_urdf/urdf/robot.xacro (robot description, xacro)
@@ -119,5 +119,5 @@
   </inertial>
   <visual>
-    <origin rpy="0 0 0" xyz="-0.641 -0.350743 -0.04081"/>
+    <origin rpy="0 0 0" xyz="-0.741 -0.350743 -0.04081"/>
     <geometry>
       <mesh filename="package://nsra_urdf/urdf/mm_stl/Component5_1.stl" scale="0.001 0.001 0.001"/>
@@ -128,5 +128,5 @@
   </visual>
   <collision>
-    <origin rpy="0 0 0" xyz="-0.641 -0.350743 -0.04081"/>
+    <origin rpy="0 0 0" xyz="-0.741 -0.350743 -0.04081"/>
     <geometry>
       <mesh filename="package://nsra_urdf/urdf/mm_stl/Component5_1.stl" scale="0.001 0.001 0.001"/>

Commit message: Update robot.xacro

File: robot_ws/src/nsra_urdf/urdf/robot.xacro (robot description, xacro)
@@ -119,5 +119,5 @@
   </inertial>
   <visual>
-    <origin rpy="0 0 0" xyz="-0.741 -0.350743 -0.04081"/>
+    <origin rpy="0 0 0" xyz="-0.541 -0.350743 -0.04081"/>
     <geometry>
       <mesh filename="package://nsra_urdf/urdf/mm_stl/Component5_1.stl" scale="0.001 0.001 0.001"/>
@@ -128,5 +128,5 @@
   </visual>
   <collision>
-    <origin rpy="0 0 0" xyz="-0.741 -0.350743 -0.04081"/>
+    <origin rpy="0 0 0" xyz="-0.541 -0.350743 -0.04081"/>
     <geometry>
       <mesh filename="package://nsra_urdf/urdf/mm_stl/Component5_1.stl" scale="0.001 0.001 0.001"/>

Commit message: Update robot.xacro

File: robot_ws/src/nsra_urdf/urdf/robot.xacro (robot description, xacro)
@@ -141,5 +141,5 @@
   </inertial>
   <visual>
-    <origin rpy="0 0 0" xyz="-0.693 -0.350743 -0.00081"/>
+    <origin rpy="0 0 0" xyz="-0.593 -0.350743 -0.00081"/>
     <geometry>
       <mesh filename="package://nsra_urdf/urdf/mm_stl/Component6_1.stl" scale="0.001 0.001 0.001"/>
@@ -150,5 +150,5 @@
   </visual>
   <collision>
-    <origin rpy="0 0 0" xyz="-0.693 -0.350743 -0.00081"/>
+    <origin rpy="0 0 0" xyz="-0.593 -0.350743 -0.00081"/>
     <geometry>
       <mesh filename="package://nsra_urdf/urdf/mm_stl/Component6_1.stl" scale="0.001 0.001 0.001"/>

Commit message: Update robot.xacro

File: robot_ws/src/nsra_urdf/urdf/robot.xacro (robot description, xacro)
@@ -163,5 +163,5 @@
   </inertial>
   <visual>
-    <origin rpy="0 0 0" xyz="0.082596 -0.148634 -0.225661"/>
+    <origin rpy="0 0 0" xyz="0.182596 -0.148634 -0.225661"/>
     <geometry>
       <mesh filename="package://nsra_urdf/urdf/mm_stl/Component8_1.stl" scale="0.001 0.001 0.001"/>
@@ -172,5 +172,5 @@
   </visual>
   <collision>
-    <origin rpy="0 0 0" xyz="0.082596 -0.148634 -0.225661"/>
+    <origin rpy="0 0 0" xyz="0.182596 -0.148634 -0.225661"/>
     <geometry>
       <mesh filename="package://nsra_urdf/urdf/mm_stl/Component8_1.stl" scale="0.001 0.001 0.001"/>
@@ -185,5 +185,5 @@
   </inertial>
   <visual>
-    <origin rpy="0 0 0" xyz="0.082596 -0.190634 -0.085661"/>
+    <origin rpy="0 0 0" xyz="0.182596 -0.190634 -0.085661"/>
     <geometry>
       <mesh filename="package://nsra_urdf/urdf/mm_stl/Component7_1.stl" scale="0.001 0.001 0.001"/>
@@ -194,5 +194,5 @@
   </visual>
   <collision>
-    <origin rpy="0 0 0" xyz="0.082596 -0.190634 -0.085661"/>
+    <origin rpy="0 0 0" xyz="0.182596 -0.190634 -0.085661"/>
     <geometry>
       <mesh filename="package://nsra_urdf/urdf/mm_stl/Component7_1.stl" scale="0.001 0.001 0.001"/>
